Commit message: started to configure husky

File: ros_gibson_environment/robot_models/husky.urdf (robot description, URDF)
Before this commit: robot husky_robot, 12 links, 11 joints
Joints:
- joint eyes_joint: origin xyz=0.4 0 1.00 rpy=1.57 0 -1.57 -> xyz=0.4 0 1.00 rpy=-1.57 0 -1.57

Commit message: fixed point cloud position

File: ros_gibson_environment/robot_models/husky.urdf (robot description, URDF)
Before this commit: robot husky_robot, 12 links, 11 joints
Links:
- added link base_footprint
Joints:
- added joint base_footprint_joint: type fixed, parent base_footprint, child base_link, origin xyz=0 0 0.13 rpy=0 0 0
- joint eyes_joint: origin xyz=0.4 0 1.00 rpy=-1.57 0 -1.57 -> xyz=0.4 0 0.6 rpy=-1.57 0 -1.57
